File: eagle/qc/qc.sch (EAGLE design)
At the start: 40 parts, among them IC1 IRFS7530, IC2 IRFS7530, IC3 IRFS7530, IC4 IRFS7530, IC5 IRFS7530, IC6 IRFS7530, U1 DRV8302

Commit message: added FETs and related circuitry for the motor drive, current sense
Parts:
- removed C1, C10, C11, C12, C2, C3, C4, C5, C6, C7, C8, C9: (no value), resistor:C-EUC0603
- removed C13, C14, C15, C16, C17: (no value), resistor:C-EUC0805
- removed IC1, IC2, IC3, IC4, IC5, IC6: IRFS7530, IRFS7530:IRFS7530
- removed R1, R2, R3, R4, R5, R6, R7, R8, R9: (no value), resistor:R-US_R0603
- removed R10: (no value), resistor:R-US_R0805
- removed U1: DRV8302, drv8302:DRV8302
